Commit message: 0130
simulation fix

File: 01_docs/robot_description/ur10_2m/robot_description.urdf (robot description, URDF)
Before this commit: robot ur10, 11 links, 10 joints
Links:
- link base_link: geometry collision mesh filename=package://robot_description/meshes/base_bachmann.stl; visual mesh filename=package://robot_description/meshes/base_bachmann.stl
- link ee_link: geometry collision mesh filename=package://robot_description/meshes/end_effector_e2e.stl; visual mesh filename=package://robot_description/meshes/end_effector_e2e.stl
